Commit message: [oakd_lite_desc] Gazebo launched, bug fixes still required

File: oakd_lite_description/urdf/oakd_lite.urdf.xacro (robot description, xacro)
@@ -1,10 +1,8 @@
 <robot xmlns:xacro="http://www.ros.org/wiki/xacro" name = "OAKD_Lite_Camera">
     <xacro:include filename="$(find oakd_lite_description)/urdf/oakd_lite.xacro" />
-    <xacro:oakd name = "oakd" parent_link = "world">
-        <origin xzy = " 0 0 0 " rpy = " 1.57 0 1.57"/>
+    <xacro:oakd name="oakd" parent_link="world">
+        <origin xzy = " 0 0 0 " rpy = " 1.57 0 -1.57"/>
     </xacro:oakd>
-    <!-- Remove World link and set above parent link to whatever link you would like to attach the camera to-->
-    <link name = "world">
-        <origin xzy = " 0 0 0 " rpy = " 0 0 0"/>
-    </link>
+    <!-- Remove World link and set above parent link to whatever link you would like to attach the camera to. Change default RVIZ framein launch file-->
+    <link name = "world"/>
 </robot>

File: oakd_lite_description/urdf/oakd_lite.xacro (robot description, xacro)
@@ -1,4 +1,4 @@
 <?xml version="1.0"?>
-<robot xmlns:xacro="http://ros.org/wiki/xacro">
+<robot xmlns:xacro="http://ros.org/wiki/xacro" name = "OAKD_Lite_Camera">
 <xacro:macro name="oakd" params="name:=oakd parent_link *origin model:=pro">
   <xacro:include filename="$(find oakd_lite_description)/urdf/common_properties.urdf.xacro"/>
@@ -24,7 +24,10 @@
         <mesh filename="file://$(find oakd_lite_description)/meshes/oakd_lite.stl" scale="1 1 1" />
       </geometry>
+      <material name = "green">
+          <color rgba = "0.0 1.0 0.0 0.8"/>
+      </material>
     </visual>
     <collision>
-      <origin xyz="${collision_offset_x} ${collision_offset_y} ${collision_offset_z}"/>
+      <origin xyz="${collision_offset_x} ${collision_offset_y} ${collision_offset_z}" rpy = "0 0 0"/>
       <geometry>
         <box size="${collision_length_x} ${collision_length_y} ${collision_length_z}"/>
@@ -32,4 +35,5 @@
     </collision>
     <inertial>
+      <origin xyz="${collision_offset_x} ${collision_offset_y} ${collision_offset_z}" rpy = "0 0 0"/>
       <mass value="${mass}"/>
       <inertia ixx="0.00000202475" ixy="0.0" ixz="0.0"
@@ -98,6 +102,11 @@
   </joint>
   <!-- Gazebo links and joints -->
+  <gazebo>
+    <plugin filename="libignition-gazebo-joint-state-publisher-system.so"
+      name="ignition::gazebo::systems::JointStatePublisher"/>
+  </gazebo>
   <gazebo reference="${name}_rgb_camera_frame">
     <sensor name="rgbd_camera" type="rgbd_camera">
+      <topic>oakd_lite</topic>
       <camera>
         <horizontal_fov>1.25</horizontal_fov>
@@ -114,6 +123,8 @@
       <update_rate>30</update_rate>
       <visualize>true</visualize>
+      <plugin filename = "ignition-gazebo-sensors-system"
+        name = "ignition::gazebo::systems::Sensors">
+      </plugin>
     </sensor>
-    <xacro:material_darkgray/>
   </gazebo>
   <gazebo reference="${name}_joint">

Commit message: [oakd_lite_desc] Functioning RVIZ and Gazebo

File: oakd_lite_description/urdf/oakd_lite.urdf.xacro (robot description, xacro)
@@ -1,8 +1,14 @@
 <robot xmlns:xacro="http://www.ros.org/wiki/xacro" name = "OAKD_Lite_Camera">
+    <!-- Remove World link and set above parent link to whatever link you would like to attach the camera to. Change default RVIZ framein launch file-->
+    <link name = "world">
+        <inertial>
+            <origin rpy="0 0 0" xyz="0 0 0"/>
+            <mass value="1"/>
+            <inertia ixx="1.0" ixy="0.0" ixz="0.0" iyy="1.0" iyz="0.0" izz="1.0"/>
+        </inertial>
+    </link>
     <xacro:include filename="$(find oakd_lite_description)/urdf/oakd_lite.xacro" />
     <xacro:oakd name="oakd" parent_link="world">
         <origin xzy = " 0 0 0 " rpy = " 1.57 0 -1.57"/>
     </xacro:oakd>
-    <!-- Remove World link and set above parent link to whatever link you would like to attach the camera to. Change default RVIZ framein launch file-->
-    <link name = "world"/>
 </robot>

File: oakd_lite_description/urdf/oakd_lite.xacro (robot description, xacro)
@@ -1,5 +1,5 @@
 <?xml version="1.0"?>
 <robot xmlns:xacro="http://ros.org/wiki/xacro" name = "OAKD_Lite_Camera">
-<xacro:macro name="oakd" params="name:=oakd parent_link *origin model:=pro">
+<xacro:macro name="oakd" params="name parent_link *origin">
   <xacro:include filename="$(find oakd_lite_description)/urdf/common_properties.urdf.xacro"/>
   <xacro:property name="mass"       value="0.061"/>
@@ -48,5 +48,5 @@
       <parent link="${base_frame}"/>
       <child link="${name}_rgb_camera_frame"/>
-      <origin xyz="0 0 0" rpy="0 0 0" />
+      <origin xyz="0 0 0" rpy="-1.57 -1.57 0" />
   </joint>
   <link name="${name}_rgb_camera_optical_frame">
