Commit message: [rplidar_a1_description] ray_sensor xacro defined here was apparently messing with other ray sensors in the create3 description

File: rplidar_a1_description/urdf/rplidar.xacro (robot description, xacro)
@@ -18,5 +18,5 @@
     </xacro:inertial_cuboid_with_pose>
   </xacro:macro>
-  <xacro:macro name="ray_sensor"
+  <xacro:macro name="rp_ray_sensor"
                params="sensor_name gazebo update_rate visualize
             h_samples h_res h_min_angle h_max_angle
@@ -129,5 +129,5 @@
   </link>
   <gazebo reference="${name}_link">
-    <xacro:ray_sensor sensor_name="${name}" gazebo="${gazebo}"
+    <xacro:rp_ray_sensor sensor_name="${name}" gazebo="${gazebo}"
                   update_rate="62.0" visualize="1"
                   h_samples="640" h_res="1.0" h_min_angle="${-pi}" h_max_angle="${pi}"
@@ -135,5 +135,5 @@
                   <plugin name="ignition::gazebo::systems::Sensors"
                           filename="libignition-gazebo-sensors-system.so"/>
-    </xacro:ray_sensor>
+    </xacro:rp_ray_sensor>
     <xacro:material_darkgray/>
   </gazebo>

Commit message: [rplidar sim] changed lidar frame to match what SLAM toolbox expects, added base_footprint fixed joint in xacro to sidestep issue spinning static transform separately

File: rplidar_a1_description/urdf/rplidar.xacro (robot description, xacro)
@@ -88,5 +88,5 @@
         </lidar>
         <xacro:insert_block name="plugin"/>
-        <ignition_frame_id>${name}_link</ignition_frame_id>
+        <ignition_frame_id>laser_frame</ignition_frame_id>
       </sensor>
     </xacro:if>
@@ -113,5 +113,5 @@
   <xacro:property name="collision_y_offset"       value="${1.3*cm2m}" />
   <xacro:property name="collision_z_offset"       value="${-1.9*cm2m}" />
-  <link name="${name}_link">
+  <link name="laser_frame">
     <visual>
       <geometry>
@@ -128,6 +128,6 @@
     <xacro:inertial_cuboid mass="0.17" x="${length_x}" y="${length_y}" z="${length_z}"/>
   </link>
-  <gazebo reference="${name}_link">
-    <xacro:rp_ray_sensor sensor_name="${name}" gazebo="${gazebo}"
+  <gazebo reference="laser_frame">
+    <xacro:rp_ray_sensor sensor_name="laser_frame" gazebo="${gazebo}"
                   update_rate="62.0" visualize="1"
                   h_samples="640" h_res="1.0" h_min_angle="${-pi}" h_max_angle="${pi}"
@@ -142,5 +142,5 @@
   <joint name="${name}_joint" type="fixed">
     <parent link="${parent_link}"/>
-    <child link="${name}_link"/>
+    <child link="laser_frame"/>
     <xacro:insert_block name="origin"/>
   </joint>
@@ -148,4 +148,10 @@
     <preserveFixedJoint>true</preserveFixedJoint>
   </gazebo>
+  <link name="base_footprint"/>
+  <joint name="base_footprint_fixed_joint" type="fixed">
+    <parent link="laser_frame"/>
+    <child link="base_footprint"/>
+    <origin xyz="0 0 0" rpy="0 0 0"/>
+  </joint>
     <gazebo>
       <plugin filename="libignition-gazebo-joint-state-publisher-system.so"
