Commit message: Empty.sdf, camera, no lidar

File: create3_sim_total/urdf/create3_total.urdf.xacro (robot description, xacro)
@@ -181,12 +181,10 @@
   </xacro:ir_intensity>
   <!-- Added Sensors -->
-  <!--
   <xacro:oakd name="oakd" parent_link="base_link">
-    <origin xzy = " 0 0 0 " rpy = " 1.57 0 -1.57"/>
+    <origin xyz = " 0 0 0.5 " rpy = " 1.57 0 -1.57"/>
   </xacro:oakd>
-  <xacro:rplidar name="rplidar" parent_link="base_link" gazebo="ignition">
+  <!-- <xacro:rplidar name="rplidar" parent_link="base_link" gazebo="ignition">
     <origin xyz="0 0 0" rpy="0 0 0"/>
-  </xacro:rplidar>
-  -->
+  </xacro:rplidar> -->
   <!-- Buttons -->
   <xacro:button
@@ -254,9 +252,10 @@
       <plugin filename="libignition-gazebo-contact-system.so" name="ignition::gazebo::systems::Contact"></plugin>
     </gazebo>
+<!--
     <gazebo>
       <plugin filename="libignition-gazebo-sensors-system.so" name="ignition::gazebo::systems::Sensors">
         <render_engine>ogre</render_engine>
       </plugin>
-    </gazebo>
+    </gazebo> -->
   </xacro:if>
 </robot>

File: oakd_lite_description/urdf/oakd_lite.urdf.xacro (robot description, xacro)
@@ -10,5 +10,5 @@
     <xacro:include filename="$(find oakd_lite_description)/urdf/oakd_lite.xacro" />
     <xacro:oakd name="oakd" parent_link="world">
-        <origin xzy = " 0 0 0 " rpy = " 1.57 0 -1.57"/>
+        <origin xyz = " 0 0 0 " rpy = " 1.57 0 -1.57"/>
     </xacro:oakd>
 </robot>

File: oakd_lite_description/urdf/oakd_lite.xacro (robot description, xacro)
@@ -125,4 +125,5 @@
       <plugin filename = "ignition-gazebo-sensors-system"
         name = "ignition::gazebo::systems::Sensors">
+        <render_engine>ogre</render_engine>
       </plugin>
     </sensor>

Commit message: Functioning Create3, camera and Lidar TOGETHER

File: create3_sim_total/urdf/create3_total.urdf.xacro (robot description, xacro)
@@ -184,7 +184,7 @@
     <origin xyz = " 0 0 0.5 " rpy = " 1.57 0 -1.57"/>
   </xacro:oakd>
-  <!-- <xacro:rplidar name="rplidar" parent_link="base_link" gazebo="ignition">
-    <origin xyz="0 0 0" rpy="0 0 0"/>
-  </xacro:rplidar> -->
+  <xacro:rplidar name="rplidar" parent_link="base_link" gazebo="ignition">
+    <origin xyz="0 0 1" rpy="0 0 0"/>
+  </xacro:rplidar>
   <!-- Buttons -->
   <xacro:button
@@ -252,8 +252,7 @@
       <plugin filename="libignition-gazebo-contact-system.so" name="ignition::gazebo::systems::Contact"></plugin>
     </gazebo>
-<!--
-    <gazebo>
+    <!-- <gazebo>
       <plugin filename="libignition-gazebo-sensors-system.so" name="ignition::gazebo::systems::Sensors">
-        <render_engine>ogre</render_engine>
+        <render_engine>ogre2</render_engine>
       </plugin>
     </gazebo> -->

File: oakd_lite_description/urdf/oakd_lite.xacro (robot description, xacro)
@@ -123,8 +123,12 @@
       <update_rate>30</update_rate>
       <visualize>true</visualize>
-      <plugin filename = "ignition-gazebo-sensors-system"
+      <!-- <plugin filename = "ignition-gazebo-sensors-system"
         name = "ignition::gazebo::systems::Sensors">
         <render_engine>ogre2</render_engine>
+<<<<<<< Updated upstream
       </plugin>
+=======
+      </plugin> -->
+>>>>>>> Stashed changes
     </sensor>
   </gazebo>

File: rplidar_a1_description/urdf/rplidar.xacro (robot description, xacro)
@@ -134,5 +134,7 @@
                   r_min="0.164" r_max="12.0" r_res="0.01">
                   <plugin name="ignition::gazebo::systems::Sensors"
-                          filename="libignition-gazebo-sensors-system.so"/>
+                          filename="libignition-gazebo-sensors-system.so">
+                    <render_engine>ogre2</render_engine>
+                  </plugin>
     </xacro:rp_ray_sensor>
     <xacro:material_darkgray/>

Commit message: [create3 xacro] updated positions of lidar and camera to roughly be realistic

File: create3_sim_total/urdf/create3_total.urdf.xacro (robot description, xacro)
@@ -182,8 +182,8 @@
   <!-- Added Sensors -->
   <xacro:oakd name="oakd" parent_link="base_link">
-    <origin xyz = " 0 0 0.5 " rpy = " 1.57 0 -1.57"/>
+    <origin xyz = " 0.06 0 0.17 " rpy = " 1.57 0 -1.57"/>
   </xacro:oakd>
   <xacro:rplidar name="rplidar" parent_link="base_link" gazebo="ignition">
-    <origin xyz="0 0 1" rpy="0 0 0"/>
+    <origin xyz="0 0 0.14" rpy="0 0 0"/>
   </xacro:rplidar>
   <!-- Buttons -->

Commit message: [sim] moved base_footprint link/joint definition to create3_sim package instead of rplidar package

File: create3_sim_total/urdf/create3_total.urdf.xacro (robot description, xacro)
@@ -187,4 +187,10 @@
     <origin xyz="0 0 0.14" rpy="0 0 0"/>
   </xacro:rplidar>
+  <link name="base_footprint"/>
+  <joint name="base_footprint_fixed_joint" type="fixed">
+    <parent link="laser_frame"/>
+    <child link="base_footprint"/>
+    <origin xyz="0 0 0" rpy="0 0 0"/>
+  </joint>
   <!-- Buttons -->
   <xacro:button

File: rplidar_a1_description/urdf/rplidar.xacro (robot description, xacro)
@@ -148,10 +148,4 @@
     <preserveFixedJoint>true</preserveFixedJoint>
   </gazebo>
-  <link name="base_footprint"/>
-  <joint name="base_footprint_fixed_joint" type="fixed">
-    <parent link="laser_frame"/>
-    <child link="base_footprint"/>
-    <origin xyz="0 0 0" rpy="0 0 0"/>
-  </joint>
     <gazebo>
       <plugin filename="libignition-gazebo-joint-state-publisher-system.so"

Commit message: [sim] updated transform between base_footprint and laser_frame to reflect static transform in create3_lidar's sensor bringup launch file

File: create3_sim_total/urdf/create3_total.urdf.xacro (robot description, xacro)
@@ -191,5 +191,5 @@
     <parent link="laser_frame"/>
     <child link="base_footprint"/>
-    <origin xyz="0 0 0" rpy="0 0 0"/>
+    <origin xyz="0.012 0 -0.144" rpy="0 0 0"/>
   </joint>
   <!-- Buttons -->
